File: Hardware/Pure Keys aec-pcb1.brd (EAGLE design)
At the start: 99 x 98.7 mm, 58 parts, among them IC1 TL074P, IC2 TL072P, IC5 TL074P, Q2 20MHz, T1 2N3904, U2 LM4040A50IDBZT, U3 328P

Commit message: changed 74238 for 74138
Parts:
- V1: value 74238N -> 74138N
Changed lines of the file:
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@@
 <attribute name="PROD_ID" value="IC-09136" x="41.91" y="58.42" size="1.778" layer="27" display="off"/>
 </element>
-<element name="V1" library="74ttl-din" library_urn="urn:adsk.eagle:library:84" package="DIL16" package3d_urn="urn:adsk.eagle:package:1462/1" value="74238N" x="34.29" y="72.39"/>
+<element name="V1" library="74ttl-din" library_urn="urn:adsk.eagle:library:84" package="DIL16" package3d_urn="urn:adsk.eagle:package:1462/1" value="74138N" x="34.29" y="72.39"/>
 <element name="V2" library="74ttl-din" library_urn="urn:adsk.eagle:library:84" package="DIL16" package3d_urn="urn:adsk.eagle:package:1462/1" value="74151N" x="72.39" y="73.66"/>
 <element name="R4" library="rcl" package="R0805" value="10K" x="20.32" y="38.1"/>
