File: Hardware/Pure Keys aec-pcb3-inProgress.sch (EAGLE design)
At the start: 61 parts, among them IC1 MCP6004P, IC5 MCP6004P, Q2 20MHz, T1 2N3904, U2 LM4040, U3 328P

Commit message: adding part numbers to attributes
Parts:
- R1, R10, R11, R12, R13: RS-PART (none) -> 223-0427
- U2: RS-PART (none) -> 809-6343
Changed lines of the file:
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@@
 <part name="U2" library="GMSN-R2Project" deviceset="LM4040A30IDBZT" device="" value="LM4040">
 <attribute name="MPN" value="LM4040A30IDBZT"/>
+<attribute name="RS-PART" value="809-6343"/>
 </part>
 <part name="R3" library="rcl" deviceset="R-US_" device="R0805" value="2K"/>
@@
 <part name="R8" library="rcl" deviceset="R-US_" device="R0805" value="100K"/>
 <part name="R9" library="rcl" deviceset="R-US_" device="R0805" value="100K"/>
-<part name="R1" library="rcl" deviceset="R-US_" device="R0805" value="1K"/>
-<part name="R10" library="rcl" deviceset="R-US_" device="R0805" value="1K"/>
-<part name="R11" library="rcl" deviceset="R-US_" device="R0805" value="1K"/>
-<part name="R12" library="rcl" deviceset="R-US_" device="R0805" value="1K"/>
-<part name="R13" library="rcl" deviceset="R-US_" device="R0805" value="1K"/>
+<part name="R1" library="rcl" deviceset="R-US_" device="R0805" value="1K">
+<attribute name="RS-PART" value="223-0427"/>
+</part>
+<part name="R10" library="rcl" deviceset="R-US_" device="R0805" value="1K">
+<attribute name="RS-PART" value="223-0427"/>
+</part>
+<part name="R11" library="rcl" deviceset="R-US_" device="R0805" value="1K">
+<attribute name="RS-PART" value="223-0427"/>
+</part>
+<part name="R12" library="rcl" deviceset="R-US_" device="R0805" value="1K">
+<attribute name="RS-PART" value="223-0427"/>
+</part>
+<part name="R13" library="rcl" deviceset="R-US_" device="R0805" value="1K">
+<attribute name="RS-PART" value="223-0427"/>
+</part>
 </parts>
 <sheets>
@@
 <instance part="C4" gate="G$1" x="43.18" y="43.18"/>
 <instance part="JP2" gate="G$1" x="25.4" y="38.1" rot="MR0"/>
-<instance part="U2" gate="A" x="119.38" y="40.64" rot="R90"/>
+<instance part="U2" gate="A" x="119.38" y="40.64" rot="R90">
+<attribute name="RS-PART" x="119.38" y="40.64" size="1.778" layer="96" rot="R90" display="off"/>
+</instance>
 <instance part="R3" gate="G$1" x="119.38" y="58.42" rot="R90"/>
 </instances>
@@
 <instance part="R22" gate="G$1" x="93.98" y="17.78" rot="R90"/>
 <instance part="U$4" gate="G$1" x="76.2" y="81.28"/>
-<instance part="R1" gate="G$1" x="-10.16" y="58.42" rot="R90"/>
-<instance part="R10" gate="G$1" x="0" y="58.42" rot="R90"/>
-<instance part="R11" gate="G$1" x="7.62" y="58.42" rot="R90"/>
-<instance part="R12" gate="G$1" x="15.24" y="58.42" rot="R90"/>
-<instance part="R13" gate="G$1" x="22.86" y="58.42" rot="R90"/>
+<instance part="R1" gate="G$1" x="-10.16" y="58.42" rot="R90">
+<attribute name="RS-PART" x="-10.16" y="58.42" size="1.778" layer="96" rot="R90" display="off"/>
+</instance>
+<instance part="R10" gate="G$1" x="0" y="58.42" rot="R90">
+<attribute name="RS-PART" x="0" y="58.42" size="1.778" layer="96" rot="R90" display="off"/>
+</instance>
+<instance part="R11" gate="G$1" x="7.62" y="58.42" rot="R90">
+<attribute name="RS-PART" x="7.62" y="58.42" size="1.778" layer="96" rot="R90" display="off"/>
+</instance>
+<instance part="R12" gate="G$1" x="15.24" y="58.42" rot="R90">
+<attribute name="RS-PART" x="15.24" y="58.42" size="1.778" layer="96" rot="R90" display="off"/>
+</instance>
+<instance part="R13" gate="G$1" x="22.86" y="58.42" rot="R90">
+<attribute name="RS-PART" x="22.86" y="58.42" size="1.778" layer="96" rot="R90" display="off"/>
+</instance>
 </instances>
 <busses>
@@
 </segment>
 <segment>
-<pinref part="R10" gate="G$1" pin="2"/>
 <wire x1="0" y1="63.5" x2="0" y2="66.04" width="0.1524" layer="91"/>
 <label x="0" y="66.04" size="1.778" layer="95"/>
+<pinref part="R10" gate="G$1" pin="2"/>
 </segment>
 </net>
@@
 </segment>
 <segment>
-<pinref part="R11" gate="G$1" pin="2"/>
 <wire x1="7.62" y1="63.5" x2="7.62" y2="66.04" width="0.1524" layer="91"/>
 <label x="7.62" y="66.04" size="1.778" layer="95"/>
+<pinref part="R11" gate="G$1" pin="2"/>
 </segment>
 </net>
@@
 </segment>
 <segment>
-<pinref part="R12" gate="G$1" pin="2"/>
 <wire x1="15.24" y1="63.5" x2="15.24" y2="66.04" width="0.1524" layer="91"/>
 <label x="15.24" y="66.04" size="1.778" layer="95"/>
+<pinref part="R12" gate="G$1" pin="2"/>
 </segment>
 </net>
@@
 </segment>
 <segment>
-<pinref part="R13" gate="G$1" pin="2"/>
 <wire x1="22.86" y1="63.5" x2="22.86" y2="66.04" width="0.1524" layer="91"/>
 <label x="22.86" y="66.04" size="1.778" layer="95"/>
+<pinref part="R13" gate="G$1" pin="2"/>
 </segment>
 </net>
@@
 <pinref part="R1" gate="G$1" pin="1"/>
 <wire x1="-10.16" y1="53.34" x2="-10.16" y2="50.8" width="0.1524" layer="91"/>
-<pinref part="R10" gate="G$1" pin="1"/>
 <wire x1="0" y1="53.34" x2="0" y2="50.8" width="0.1524" layer="91"/>
 <wire x1="-10.16" y1="50.8" x2="0" y2="50.8" width="0.1524" layer="91"/>
-<pinref part="R11" gate="G$1" pin="1"/>
 <wire x1="7.62" y1="53.34" x2="7.62" y2="50.8" width="0.1524" layer="91"/>
 <wire x1="0" y1="50.8" x2="7.62" y2="50.8" width="0.1524" layer="91"/>
 <junction x="0" y="50.8"/>
-<pinref part="R12" gate="G$1" pin="1"/>
 <wire x1="15.24" y1="53.34" x2="15.24" y2="50.8" width="0.1524" layer="91"/>
 <wire x1="7.62" y1="50.8" x2="15.24" y2="50.8" width="0.1524" layer="91"/>
 <junction x="7.62" y="50.8"/>
-<pinref part="R13" gate="G$1" pin="1"/>
 <wire x1="22.86" y1="53.34" x2="22.86" y2="50.8" width="0.1524" layer="91"/>
 <wire x1="15.24" y1="50.8" x2="22.86" y2="50.8" width="0.1524" layer="91"/>
@@
 <wire x1="-17.78" y1="50.8" x2="-17.78" y2="48.26" width="0.1524" layer="91"/>
 <label x="-17.78" y="48.26" size="1.778" layer="95"/>
-</segment>
-</net>
+<pinref part="R10" gate="G$1" pin="1"/>
+<pinref part="R11" gate="G$1" pin="1"/>
+<pinref part="R12" gate="G$1" pin="1"/>
+<pinref part="R13" gate="G$1" pin="1"/>
+</segment>
+</net>

Commit message: routing on pcb-3-inprogress
Parts:
- U$4: device SparkFun-Connectors:M10X22X10_LOCK -> SparkFun-Connectors:CONN_10X2; RS-PART (none) -> 669-5364
Changed lines of the file:
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@@
 <part name="R21" library="rcl" deviceset="R-US_" device="R0805" value="10K"/>
 <part name="R22" library="rcl" deviceset="R-US_" device="R0805" value="10K"/>
-<part name="U$4" library="SparkFun-Connectors" deviceset="M10X2" device="2X10_LOCK" value="KeyBoard Connector"/>
+<part name="U$4" library="SparkFun-Connectors" deviceset="CONN_10X2" device="" value="KeyBoard Connector">
+<attribute name="RS-PART" value="669-5364"/>
+</part>
 <part name="TRIG2" library="GMSN" deviceset="PJ302M" device="" value="PJ302M"/>
 <part name="TRIG3" library="GMSN" deviceset="PJ302M" device="" value="PJ302M"/>
@@
 <instance part="R21" gate="G$1" x="81.28" y="17.78" rot="R90"/>
 <instance part="R22" gate="G$1" x="93.98" y="17.78" rot="R90"/>
-<instance part="U$4" gate="G$1" x="76.2" y="81.28"/>
+<instance part="U$4" gate="G$1" x="76.2" y="81.28">
+<attribute name="RS-PART" x="76.2" y="81.28" size="1.778" layer="96" display="off"/>
+</instance>
 <instance part="R1" gate="G$1" x="-10.16" y="58.42" rot="R90">
 <attribute name="RS-PART" x="-10.16" y="58.42" size="1.778" layer="96" rot="R90" display="off"/>
